File: electronics/syringe_pump_controller_module/syringe_pump.kicad_sch (KiCad schematic)
At the start: 68 parts, among them J1 IN, J10 EndSwitch, J11 EndSwitch, J12 Conn_01x04, J13 Conn_01x08, J2 ON OFF, J4 HDR-4x1, J5 HDR-4x1, J6 EndSwitch, J7 EndSwitch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

Commit message: v2 of module version. fixing minor bugs and redistribute components on the board
Parts:
- removed F2: FUSE, Fuse:Fuse_1206_3216Metric, symbol IoWLabs:FUSE
- added F1: FUSE, Fuse:Fuse_1206_3216Metric, symbol IoWLabs:FUSE
- added J3: HDR-3x1, Connector_BarrelJack:BarrelJack_Horizontal, symbol IoWLabsConnectors:HDR-3x1
- J1: value IN -> VIN
Connections:
- net +3V3: no longer J12.2 (Pin_2)
- net +5V: now also J12.2 (Pin_2)
- net GND: now also J3.2
- net M1_DIR: now also U7.27 (GPIO16); no longer U7.28 (GPIO17)
- net M1_STEP: now also U7.26 (ADC2_CH0/GPIO4); no longer U7.30 (GPIO18)
- net M2_DIR: now also U7.30 (GPIO18); no longer U7.26 (ADC2_CH0/GPIO4)
- net M2_STEP: now also U7.28 (GPIO17); no longer U7.27 (GPIO16)
- net M3_DIR: now also U7.9 (DAC_1/ADC2_CH8/GPIO25); no longer U7.8 (32K_XN/GPIO33/ADC1_CH5)
- net M3_EN: now also U3.11 (IO0_7); no longer U3.4 (IO0_0)
- net M3_ES: now also U3.8 (IO0_4); no longer U3.7 (IO0_3)
- net M3_MS1: now also U3.10 (IO0_6); no longer U3.5 (IO0_1)
- net M3_MS2: now also U3.9 (IO0_5); no longer U3.6 (IO0_2)
- net M3_STEP: now also U7.10 (DAC_2/ADC2_CH9/GPIO26); no longer U7.7 (32K_XP/GPIO32/ADC1_CH4)
- net M4_DIR: now also U7.7 (32K_XP/GPIO32/ADC1_CH4); no longer U7.10 (DAC_2/ADC2_CH9/GPIO26)
- net M4_EN: now also U3.7 (IO0_3); no longer U3.8 (IO0_4)
- net M4_ES: now also U3.4 (IO0_0); no longer U3.11 (IO0_7)
- net M4_MS1: now also U3.6 (IO0_2); no longer U3.9 (IO0_5)
- net M4_MS2: now also U3.5 (IO0_1); no longer U3.10 (IO0_6)
- net M4_STEP: now also U7.8 (32K_XN/GPIO33/ADC1_CH5); no longer U7.9 (DAC_1/ADC2_CH8/GPIO25)
- net SCL: now also U3.22 (SCL); no longer U3.23 (SDA)
- net SDA: now also U3.23 (SDA); no longer U3.22 (SCL)
- net VIN_12V: now also F1.2
- net VIN: now reaches J1.2
- net VIN: now also F1.1, J3.1
Other:
- note added: "01/2025"
- note added: "syringe pump BOARD - V2"
- note removed: "07/2023"
- note removed: "syringe pump BOARD"
